File: LLU/Sonar-Module/Board/RoboDiscovery-F4_v1.0/RoboDiscovery-F4_V1.0.sch (EAGLE design)
At the start: 212 parts, among them CN1 10.8060.0008, CN2 10.8060.0008, CN3 SATA-7, CN4 SATA-7, IC1 74HC4067DB, IC1B 74HC4067DB, IC2 74HC4067DB, IC2B 74HC4067DB, IC3 ULN2804A, IC4 ST3232CN, J1 J2541405-R, J2 J2541405-R, P1 PULS6X6SMD, P2 PULS6X6SMD, Q1 BC327-40, Q2 BC327-40, Q3 BC327-40, Q4 BC327-40, Q5 BC327-40, Q6 BC327-40, U1 L78XXAB/AC, U2 LD1117V33, U3 SN65176BD, X1 DB9 femmina

Commit message: RoboDiscovery-F4 V1.0 files
Connections:
- removed net +24V: POW-6.S
- net +5V/1: now also POW-6.S
- net A1: now also ENC_1-4.S, R57.1, R60.2; no longer ENC_2-4.S, R66.1, R69.2
- net A2: now also ENC_2-4.S, R66.1, R69.2; no longer ENC_1-4.S, R57.1, R60.2
- net B1: now also ENC_1-3.S, R58.1, R61.2; no longer ENC_2-3.S, R67.1, R70.2
- net B2: now also ENC_2-3.S, R67.1, R70.2; no longer ENC_1-3.S, R58.1, R61.2
- net F4_UART2_DIR: now also DIS1G$1.PC5; no longer DIS1G$1.PA0
- net I1: now also ENC_1-2.S, R59.1, R62.2; no longer ENC_2-2.S, R68.1, R71.2
- net I2: now also ENC_2-2.S, R68.1, R71.2; no longer ENC_1-2.S, R59.1, R62.2
Changed lines of the file:
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@@
 <?xml version="1.0" encoding="utf-8"?>
 <!DOCTYPE eagle SYSTEM "eagle.dtd">
-<eagle version="6.4">
+<eagle version="6.5.0">
 <drawing>
 <settings>
@@
 <part name="POW" library="con-molex" deviceset="22-?-06" device="27-2061" value="J2541406-R"/>
 <part name="GND93" library="supply1" deviceset="GND" device=""/>
-<part name="P+28" library="supply1" deviceset="+24V" device=""/>
 <part name="P+29" library="supply1" deviceset="+5V" device=""/>
 <part name="+3V17" library="supply1" deviceset="+3V3" device=""/>
@@
 <part name="+3V7" library="supply1" deviceset="+3V3" device=""/>
 <part name="+3V9" library="supply1" deviceset="+3V3" device=""/>
+<part name="SUPPLY45" library="supply2" deviceset="+5V/1" device=""/>
 </parts>
 <sheets>
@@
 <net name="F4_UART2_DIR" class="0">
 <segment>
-<wire x1="88.9" y1="121.92" x2="93.98" y2="121.92" width="0.1524" layer="91"/>
-<label x="93.98" y="121.92" size="1.27" layer="95" xref="yes"/>
-<pinref part="DIS1" gate="G$1" pin="PA0"/>
+<wire x1="58.42" y1="111.76" x2="53.34" y2="111.76" width="0.1524" layer="91"/>
+<label x="53.34" y="111.76" size="1.27" layer="95" rot="R180" xref="yes"/>
+<pinref part="DIS1" gate="G$1" pin="PC5"/>
 </segment>
 </net>
@@
 <attribute name="VALUE" x="243.84" y="30.48" size="1.4224" layer="96" font="vector" ratio="10"/>
 </instance>
-<instance part="P+28" gate="1" x="238.76" y="66.04" smashed="yes" rot="R90">
-<attribute name="VALUE" x="243.84" y="63.5" size="1.4224" layer="96" font="vector" ratio="10" rot="R180"/>
-</instance>
 <instance part="P+29" gate="1" x="236.22" y="55.88" smashed="yes" rot="R90">
 <attribute name="VALUE" x="241.3" y="53.34" size="1.4224" layer="96" font="vector" ratio="10" rot="R180"/>
@@
 <attribute name="VALUE" x="162.56" y="33.02" size="1.4224" layer="96" font="vector" ratio="10"/>
 </instance>
+<instance part="SUPPLY45" gate="G$1" x="238.76" y="66.04" smashed="yes" rot="R90">
+<attribute name="VALUE" x="235.585" y="62.865" size="1.778" layer="96" rot="R90"/>
+</instance>
 </instances>
 <busses>
@@
 </segment>
 </net>
-<net name="+24V" class="0">
-<segment>
-<wire x1="241.3" y1="66.04" x2="248.92" y2="66.04" width="0.1524" layer="91"/>
-<pinref part="P+28" gate="1" pin="+24V"/>
-<pinref part="POW" gate="-6" pin="S"/>
-</segment>
-</net>
-<net name="A1" class="0">
+<net name="A2" class="0">
 <segment>
 <wire x1="109.22" y1="66.04" x2="121.92" y2="66.04" width="0.1524" layer="91"/>
@@
 </segment>
 </net>
-<net name="B1" class="0">
+<net name="B2" class="0">
 <segment>
 <wire x1="109.22" y1="60.96" x2="124.46" y2="60.96" width="0.1524" layer="91"/>
@@
 </segment>
 </net>
-<net name="I1" class="0">
+<net name="I2" class="0">
 <segment>
 <wire x1="109.22" y1="55.88" x2="127" y2="55.88" width="0.1524" layer="91"/>
@@
 </segment>
 </net>
-<net name="A2" class="0">
+<net name="A1" class="0">
 <segment>
 <wire x1="30.48" y1="66.04" x2="38.1" y2="66.04" width="0.1524" layer="91"/>
@@
 </segment>
 </net>
-<net name="B2" class="0">
+<net name="B1" class="0">
 <segment>
 <wire x1="30.48" y1="60.96" x2="40.64" y2="60.96" width="0.1524" layer="91"/>
@@
 </segment>
 </net>
-<net name="I2" class="0">
+<net name="I1" class="0">
 <segment>
 <wire x1="30.48" y1="55.88" x2="43.18" y2="55.88" width="0.1524" layer="91"/>
@@
 </segment>
 </net>
+<net name="+5V/1" class="0">
+<segment>
+<pinref part="SUPPLY45" gate="G$1" pin="+5V/1"/>
+<pinref part="POW" gate="-6" pin="S"/>
+<wire x1="241.3" y1="66.04" x2="248.92" y2="66.04" width="0.1524" layer="91"/>
+</segment>
+</net>
